File: PCB/Eagle Files/AtoVproject 16n V1.1.brd (EAGLE design)
At the start: 248.9 x 108 mm, 176 parts, among them IC1 NCS2007, IC10 TEENSY_3.2_PIN, IC2 NCS2007, IC3 NCS2007, IC4 NCS2007, IC5 MCP6004_SMD, IC6 MCP6004_SMD, IC7 MCP6004_SMD, IC8 MCP6004_SMD, IC9 CD74HC4067SM96, J1 THONKICONN, J10 THONKICONN, J11 THONKICONN, J12 THONKICONN, J13 THONKICONN, J14 THONKICONN, J15 THONKICONN, J16 THONKICONN, J2 THONKICONN, J3 THONKICONN, J4 THONKICONN, J5 THONKICONN, J6 THONKICONN, J7 THONKICONN, J8 THONKICONN, J9 THONKICONN

Commit message: Add files via upload
Parts:
- C1: value 10n -> 2.2uf
- C2: value 1u -> 1uf
- C3: value 10n -> 10nf
Changed lines of the file:
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@@
 <attribute name="VALUE" x="0.6324625" y="92.075" size="1.27" layer="27"/>
 </element>
-<element name="C3" library="rcl" library_urn="urn:adsk.eagle:library:334" package="C0805" package3d_urn="urn:adsk.eagle:package:23617/2" value="10n" x="2.54" y="85.0874625" smashed="yes" rot="R270">
+<element name="C3" library="rcl" library_urn="urn:adsk.eagle:library:334" package="C0805" package3d_urn="urn:adsk.eagle:package:23617/2" value="10nf" x="2.54" y="85.0874625" smashed="yes" rot="R270">
 <attribute name="NAME" x="3.81" y="86.3574625" size="1.27" layer="25" rot="R270"/>
 <attribute name="SPICEPREFIX" value="C" x="2.54" y="85.0874625" size="1.778" layer="27" rot="R270" display="off"/>
 <attribute name="VALUE" x="0" y="86.3574625" size="1.27" layer="27" rot="R270"/>
 </element>
-<element name="C2" library="rcl" library_urn="urn:adsk.eagle:library:334" package="C0805" package3d_urn="urn:adsk.eagle:package:23617/2" value="1u" x="2.54" y="95.2525375" smashed="yes" rot="R180">
+<element name="C2" library="rcl" library_urn="urn:adsk.eagle:library:334" package="C0805" package3d_urn="urn:adsk.eagle:package:23617/2" value="1uf" x="2.54" y="95.2525375" smashed="yes" rot="R180">
 <attribute name="NAME" x="3.81" y="93.9825375" size="1.27" layer="25" rot="R180"/>
 <attribute name="SPICEPREFIX" value="C" x="2.54" y="95.2525375" size="1.778" layer="27" rot="R180" display="off"/>
 <attribute name="VALUE" x="3.81" y="97.7925375" size="1.27" layer="27" rot="R180"/>
 </element>
-<element name="C1" library="rcl" library_urn="urn:adsk.eagle:library:334" package="C0805" package3d_urn="urn:adsk.eagle:package:23617/2" value="10n" x="2.54" y="99.0574625" smashed="yes">
-<attribute name="NAME" x="2.54" y="99.0574625" size="1.27" layer="25"/>
+<element name="C1" library="rcl" library_urn="urn:adsk.eagle:library:334" package="C0805" package3d_urn="urn:adsk.eagle:package:23617/2" value="2.2uf" x="2.54" y="99.0574625" smashed="yes">
+<attribute name="NAME" x="2.54" y="100.3274625" size="1.27" layer="25"/>
 <attribute name="SPICEPREFIX" value="C" x="2.54" y="99.0574625" size="1.778" layer="27" display="off"/>
 <attribute name="VALUE" x="1.27" y="96.5174625" size="1.27" layer="27"/>
