File: PCB/Eagle Files/AtoVproject 16n V1.1.sch (EAGLE design)
At the start: 174 parts, among them IC1 NCS2007, IC10 TEENSY_3.2_PIN, IC2 NCS2007, IC3 NCS2007, IC4 NCS2007, IC5 MCP6004_SMD, IC6 MCP6004_SMD, IC7 MCP6004_SMD, IC8 MCP6004_SMD, IC9 CD74HC4067SM96, J1 THONKICONN, J10 THONKICONN, J11 THONKICONN, J12 THONKICONN, J13 THONKICONN, J14 THONKICONN, J15 THONKICONN, J16 THONKICONN, J2 THONKICONN, J3 THONKICONN, J4 THONKICONN, J5 THONKICONN, J6 THONKICONN, J7 THONKICONN, J8 THONKICONN, J9 THONKICONN

Commit message: Add files via upload
Parts:
- C1: value 10n -> 2.2uf
- C2: value 1u -> 1uf
- C3: value 10n -> 10nf
Changed lines of the file:
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@@
 <part name="C101" library="resistor" library_urn="urn:adsk.eagle:library:348" deviceset="CPOL-EU" device="E2.5-6" package3d_urn="urn:adsk.eagle:package:23349/1" value="47uf"/>
 <part name="V1" library="v-reg-3" deviceset="LP2985" device="M5"/>
-<part name="C3" library="rcl" library_urn="urn:adsk.eagle:library:334" deviceset="C-EU" device="C0805" package3d_urn="urn:adsk.eagle:package:23617/2" value="10n"/>
-<part name="C2" library="rcl" library_urn="urn:adsk.eagle:library:334" deviceset="C-EU" device="C0805" package3d_urn="urn:adsk.eagle:package:23617/2" value="1u"/>
-<part name="C1" library="rcl" library_urn="urn:adsk.eagle:library:334" deviceset="C-EU" device="C0805" package3d_urn="urn:adsk.eagle:package:23617/2" value="10n"/>
+<part name="C3" library="rcl" library_urn="urn:adsk.eagle:library:334" deviceset="C-EU" device="C0805" package3d_urn="urn:adsk.eagle:package:23617/2" value="10nf"/>
+<part name="C2" library="rcl" library_urn="urn:adsk.eagle:library:334" deviceset="C-EU" device="C0805" package3d_urn="urn:adsk.eagle:package:23617/2" value="1uf"/>
+<part name="C1" library="rcl" library_urn="urn:adsk.eagle:library:334" deviceset="C-EU" device="C0805" package3d_urn="urn:adsk.eagle:package:23617/2" value="2.2uf"/>
 <part name="SUPPLY69" library="supply2" library_urn="urn:adsk.eagle:library:372" deviceset="+5V" device=""/>
 <part name="GND26" library="supply1" deviceset="GND" device=""/>
